File: hardware/kicad/recorder/power.kicad_sch (KiCad schematic)
At the start: 16 parts, among them U3 MCP73831-2-OT, U4 AP2112K-3.3, U5 AP22804AW5, U8 LP5907MFX-3.3

Commit message: Route the recorder board and make the fab package match it
The board had planes but no signals. It now carries 694 traces and 193
vias from freerouting, driven headless through Specctra DSN/SES, with the
USB pair, the ES8311 fanout and the analog island hand-routed first and
locked so rip-up cannot cut them.

kicad-cli pcb drc now reports zero violations at every severity and zero
unconnected items.

Two things that would have scrapped a real order:

- check_gates.py re-exported Gerbers but left the drill file, the
  pick-and-place CSV and recorder-jlc.zip at whatever date they were
  committed with. The drill file on disk predated routing and had no
  0.3 mm tool, so the package described a board with none of its vias
  drilled. The whole package is now written in one pass from one board
  file, gated on a real kicad-cli pcb drc run.
- check_placement.py trusted BOX2I.Merge()'s return value, which is an
  unrelated proxy in the SWIG bindings, and measured courtyards from
  GetCourtyard(), which is inflated past the drawn outline. That invented
  four off-board mounting holes and six overlaps. It reads the drawn
  shapes now, and check_gates runs it when pcbnew is importable.

Silkscreen designators are shrunk to the 0.8 mm / 0.15 mm fab floor and
re-seated on a full angular sweep, clearing all 29 silk warnings.

Co-authored-by: zeeman <zeeman-effect@users.noreply.github.com>
Parts:
- BT1: footprint Connector_Wire:SolderWire-2.0sqmm_1x02_D2.0mm_OD5mm -> Connector_Wire:SolderWire-2sqmm_1x02_P7.8mm_D2mm_OD3.9mm
Connections:
- net VBAT: now also C5.1
