File: hardware/kicad/recorder/power.kicad_sch (KiCad schematic)
At the start: 21 parts, among them U3 BQ24074RGTR, U4 AP2112K-3.3, U5 AP22804AW5, U8 LP5907MFX-3.3

Commit message: Keep J1 off SMT and fix MK1 pinout plus the 2.8 V analog rail.
J1 is a vertical 1x4 that will not fit under the lid, and the tails poke
toward the phone. Flag it exclude_from_bom so JLCPCB does not wave-solder
it. Keep C124378 in docs/bom.md and write jlcpcb_extra.csv so the header
can still be ordered as loose extra parts.

IM73A135 pin 3 is OUT-, a ~250 ohm amplifier output, not GND. Leave it
open; C15 still AC-couples OUT+ and C16 still takes codec MIC_N to AGND.
U8 is now LP5907-2.8 (C186700) because the capsule VDD abs max is 3.0 V.
ES8311 AVDD is 1.7-3.6 V and Y1 is 1.71-3.63 V, so the analog island can
sit at 2.8 V. Digital IO stays on VDD33.

Co-authored-by: zachrobertson19 <zachrobertson19@gmail.com>
Parts:
- U8: value LP5907MFX-3.3 -> LP5907MFX-2.8
Changed lines of the file:
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@@
 		(property "Reference" "U8" (at 80.00 197.00 0)
 			(effects (font (size 1.27 1.27))))
-		(property "Value" "LP5907MFX-3.3" (at 80.00 199.50 0)
+		(property "Value" "LP5907MFX-2.8" (at 80.00 199.50 0)
 			(effects (font (size 1.27 1.27))))
 		(property "Footprint" "Package_TO_SOT_SMD:SOT-23-5" (at 80.00 205.00 0)
