File: hardware/kicad/recorder/io.kicad_sch (KiCad schematic)
At the start: 9 parts, among them J3 microSD, SW1 record

Commit message: Route the recorder board and make the fab package match it
The board had planes but no signals. It now carries 694 traces and 193
vias from freerouting, driven headless through Specctra DSN/SES, with the
USB pair, the ES8311 fanout and the analog island hand-routed first and
locked so rip-up cannot cut them.

kicad-cli pcb drc now reports zero violations at every severity and zero
unconnected items.

Two things that would have scrapped a real order:

- check_gates.py re-exported Gerbers but left the drill file, the
  pick-and-place CSV and recorder-jlc.zip at whatever date they were
  committed with. The drill file on disk predated routing and had no
  0.3 mm tool, so the package described a board with none of its vias
  drilled. The whole package is now written in one pass from one board
  file, gated on a real kicad-cli pcb drc run.
- check_placement.py trusted BOX2I.Merge()'s return value, which is an
  unrelated proxy in the SWIG bindings, and measured courtyards from
  GetCourtyard(), which is inflated past the drawn outline. That invented
  four off-board mounting holes and six overlaps. It reads the drawn
  shapes now, and check_gates runs it when pcbnew is importable.

Silkscreen designators are shrunk to the 0.8 mm / 0.15 mm fab floor and
re-seated on a full angular sweep, clearing all 29 silk warnings.

Co-authored-by: zeeman <zeeman-effect@users.noreply.github.com>
Parts:
- SW1: footprint Button_Switch_SMD:SW_SPST_PTS645 -> Button_Switch_SMD:SW_SPST_PTS645Sx43SMTR92

Commit message: Swap SW1 for a side-actuated switch so the case needs no lever
The record button is on the left long wall, but SW1 was a top-actuated
PTS645: the plunger pointed at the phone, not at the wall. Every version of
that ends in a moulded lever inside a 9 mm stack, pivoting a sideways press
into a downward one, with the travel budget of a 3D print.

Panasonic EVQP7C01P instead. Side push, SPST, 3.5 x 2.9 x 1.35 mm, 2.2 N,
0.2 mm travel, reflow, JLCPCB C388883 and in stock. KiCad 10 already ships
the land as Button_Switch_SMD:SW_SPST_EVQP7C, and its two moulded bosses
drop into 0.7 mm NPTH holes that take the sideways load instead of the
solder joints. Rotated 270 and pushed out to x = -29.3, the actuator tip
stops 0.6 mm inside the board edge with copper still 1.46 mm off the cut.

Pin 1 now carries BTN and pin 2 GND, the other way round from the old part.
A push button's terminals are interchangeable, and after the rotation pin 2
is the pad row nearest the edge, where the F.Cu GND pour reaches it with no
trace at all; BTN gets the inner row, which has room to leave the part. The
LED via moved up to (-27.30, 16.00) and its B.Cu descent shifted to
x = -27.30 to clear the new footprint and its guide holes.

The case aperture was 7.0 x 3.5 mm, sized for "whatever mechanism this ends
up needing". It is now a 3.0 x 2.2 mm press-through slot over a 1.7 mm
actuator. The case still owes a short moulded nub to span the 0.9 mm from
the inner wall face to the actuator tip.

docs/bom.md called SW1 "side-fire, C318885". C318885 is an XKB
TS-1187A-C-J-B, a 5.1 x 5.1 x 5 mm top-actuated switch, so that line was
wrong about the part and about the direction it fires.

Board re-verified: kicad-cli pcb drc reports 0 violations at every severity,
0 unconnected items and the same 27 expected schematic-parity notes.

Co-authored-by: zeeman <zeeman-effect@users.noreply.github.com>
Parts:
- SW1: footprint Button_Switch_SMD:SW_SPST_PTS645Sx43SMTR92 -> Button_Switch_SMD:SW_SPST_EVQP7C
Connections:
- net BTN: now also SW1.1; no longer SW1.2
- net GND: now also SW1.2; no longer SW1.1
Changed lines of the file:
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@@
 		(property "Value" "record" (at 80.00 154.50 0)
 			(effects (font (size 1.27 1.27))))
-		(property "Footprint" "Button_Switch_SMD:SW_SPST_PTS645Sx43SMTR92" (at 80.00 160.00 0)
+		(property "Footprint" "Button_Switch_SMD:SW_SPST_EVQP7C" (at 80.00 160.00 0)
 			(effects (font (size 1.27 1.27)) hide))
 		(property "Datasheet" "~" (at 80.00 160.00 0)
@@
 		(stroke (width 0) (type default))
 	)
-	(global_label "GND"
+	(global_label "BTN"
 		(shape input)
 		(at 67.30 160.00 180)
@@
 		(stroke (width 0) (type default))
 	)
-	(global_label "BTN"
+	(global_label "GND"
 		(shape input)
 		(at 92.70 160.00 0)
