File: hardware/kicad/recorder/audio.kicad_sch (KiCad schematic)
At the start: 20 parts, among them U2 ES8311, U6 NS4150B, Y1 12.288MHz

Commit message: Route the recorder board and make the fab package match it
The board had planes but no signals. It now carries 694 traces and 193
vias from freerouting, driven headless through Specctra DSN/SES, with the
USB pair, the ES8311 fanout and the analog island hand-routed first and
locked so rip-up cannot cut them.

kicad-cli pcb drc now reports zero violations at every severity and zero
unconnected items.

Two things that would have scrapped a real order:

- check_gates.py re-exported Gerbers but left the drill file, the
  pick-and-place CSV and recorder-jlc.zip at whatever date they were
  committed with. The drill file on disk predated routing and had no
  0.3 mm tool, so the package described a board with none of its vias
  drilled. The whole package is now written in one pass from one board
  file, gated on a real kicad-cli pcb drc run.
- check_placement.py trusted BOX2I.Merge()'s return value, which is an
  unrelated proxy in the SWIG bindings, and measured courtyards from
  GetCourtyard(), which is inflated past the drawn outline. That invented
  four off-board mounting holes and six overlaps. It reads the drawn
  shapes now, and check_gates runs it when pcbnew is importable.

Silkscreen designators are shrunk to the 0.8 mm / 0.15 mm fab floor and
re-seated on a full angular sweep, clearing all 29 silk warnings.

Co-authored-by: zeeman <zeeman-effect@users.noreply.github.com>
Parts:
- MK1: footprint Sensor_Audio:Infineon_PG-LLGA-5-3 -> PSV:IM73A135_PG-LLGA-5-3
- SP1: footprint Speaker_Audio:Speaker_15x11mm -> PSV:Speaker_15x11mm
- U2: footprint Package_DFN_QFN:QFN-20-1EP_3x3mm_P0.4mm -> Package_DFN_QFN:QFN-20-1EP_3x3mm_P0.4mm_EP1.65x1.65mm
Connections:
- net AGND: now also U2.21 (EP)

Commit message: Pick a JLCPCB-placeable KELIKING speaker for SP1
The 15x11 placeholder could not go on the SMT line. The KLJ-01304T land, shifted pouch, and lid grille let JLC place C18186315 on a DRC-clean board.
Parts:
- SP1: value 1511 -> KLJ-01304T-08R07W; footprint PSV:Speaker_15x11mm -> PSV:Speaker_KLJ-01304T
Changed lines of the file:
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@@
 		(property "Reference" "SP1" (at 250.00 82.00 0)
 			(effects (font (size 1.27 1.27))))
-		(property "Value" "1511" (at 250.00 84.50 0)
+		(property "Value" "KLJ-01304T-08R07W" (at 250.00 84.50 0)
 			(effects (font (size 1.27 1.27))))
-		(property "Footprint" "PSV:Speaker_15x11mm" (at 250.00 90.00 0)
+		(property "Footprint" "PSV:Speaker_KLJ-01304T" (at 250.00 90.00 0)
 			(effects (font (size 1.27 1.27)) hide))
 		(property "Datasheet" "~" (at 250.00 90.00 0)
