File: hardware/kicad/recorder/audio.kicad_sch (KiCad schematic)
At the start: 20 parts, among them U2 ES8311, U6 NS4150B, Y1 12.288MHz

Commit message: Swap in a BQ24074 power-path charger so USB can run the board with the pouch unplugged.
Co-authored-by: Cursor <cursoragent@cursor.com>
Connections:
- net VBAT: no longer U6.6 (VCC)
- new net VSYS: U6.6 (VCC)
Changed lines of the file:
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@@
 		(stroke (width 0) (type default))
 	)
-	(global_label "VBAT"
+	(global_label "VSYS"
 		(shape input)
 		(at 200.00 72.22 90)
@@
 	)
 	(symbol
+		(lib_id "PSV:VSYS")
+		(at 250.00 35.00 0)
+		(unit 1)
+		(exclude_from_sim no)
+		(in_bom yes)
+		(on_board yes)
+		(dnp no)
+		(property "Reference" "#PWR13" (at 250.00 27.00 0)
+			(effects (font (size 1.27 1.27))))
+		(property "Value" "VSYS" (at 250.00 29.50 0)
+			(effects (font (size 1.27 1.27))))
+		(property "Footprint" "" (at 250.00 35.00 0)
+			(effects (font (size 1.27 1.27)) hide))
+		(property "Datasheet" "~" (at 250.00 35.00 0)
+			(effects (font (size 1.27 1.27)) hide))
+		(pin "1")
+	)
+	(wire
+		(pts (xy 250.00 35.00) (xy 250.00 42.62))
+		(stroke (width 0) (type default))
+	)
+	(global_label "VSYS"
+		(shape input)
+		(at 250.00 42.62 270)
+		(effects (font (size 1.27 1.27)) (justify right))
+	)
+	(symbol
 		(lib_id "power:PWR_FLAG")
 		(at 105.00 200.00 0)
@@
 		(property "Reference" "#FLG10" (at 105.00 192.00 0)
 			(effects (font (size 1.27 1.27))))
-		(property "Value" "pwr" (at 105.00 194.50 0)
+		(property "Value" "PWR_FLAG" (at 105.00 194.50 0)
 			(effects (font (size 1.27 1.27))))
 		(property "Footprint" "" (at 105.00 200.00 0)
