File: hardware/kicad/recorder/recorder.kicad_pcb (KiCad board)
At the start: 4 copper layers, 64 x 86 mm, 67 parts, among them J1 UART0, J2 USB_C_16P, J3 microSD, SW1 record, U1 ESP32-S3-MINI-1U-N8, U2 ES8311, U3 BQ24074RGTR, U4 AP2112K-3.3, U5 AP22804AW5, U6 NS4150B, U7 USBLC6-2SC6, U8 LP5907MFX-3.3, Y1 12.288MHz

Commit message: Keep J1 off SMT and fix MK1 pinout plus the 2.8 V analog rail.
J1 is a vertical 1x4 that will not fit under the lid, and the tails poke
toward the phone. Flag it exclude_from_bom so JLCPCB does not wave-solder
it. Keep C124378 in docs/bom.md and write jlcpcb_extra.csv so the header
can still be ordered as loose extra parts.

IM73A135 pin 3 is OUT-, a ~250 ohm amplifier output, not GND. Leave it
open; C15 still AC-couples OUT+ and C16 still takes codec MIC_N to AGND.
U8 is now LP5907-2.8 (C186700) because the capsule VDD abs max is 3.0 V.
ES8311 AVDD is 1.7-3.6 V and Y1 is 1.71-3.63 V, so the analog island can
sit at 2.8 V. Digital IO stays on VDD33.

Co-authored-by: zachrobertson19 <zachrobertson19@gmail.com>
Parts:
- U8: value LP5907MFX-3.3 -> LP5907MFX-2.8
Connections:
- MK1 pad 3: /Audio/AGND -> unconnected-(MK1-OUT--Pad3)
Routing:
- net /Audio/AGND: track 44.2 -> 43.1 mm
Changed lines of the file:
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@@
 			)
 		)
-		(attr through_hole exclude_from_pos_files)
+		(attr through_hole exclude_from_pos_files exclude_from_bom)
 		(duplicate_pad_numbers_are_jumpers no)
 		(fp_line
@@
 			)
 		)
-		(property "Value" "LP5907MFX-3.3"
+		(property "Value" "LP5907MFX-2.8"
 			(at 0 2.4 0)
 			(layer "F.Fab")
@@
 			(layers "F.Cu" "F.Mask")
 			(roundrect_rratio 0.25)
-			(net "/Audio/AGND")
+			(net "unconnected-(MK1-OUT--Pad3)")
+			(zone_connect 0)
 		)
 		(pad "4" smd roundrect
@@
 	)
 	(segment
-		(start 30.5202 11.8298)
-		(end 30.85 11.5)
-		(width 0.15)
-		(locked yes)
-		(layer "F.Cu")
-		(net "/Audio/AGND")
-	)
-	(segment
 		(start 20.9795 20)
 		(end 20.4814 20.4981)
@@
 		(width 0.15)
 		(locked yes)
-		(layer "F.Cu")
-		(net "/Audio/AGND")
-	)
-	(segment
-		(start 30.85 10.8)
-		(end 30.85 11.5)
-		(width 0.15)
-		(locked yes)

Commit message: Refresh Gerbers after lifting MK1 OUT- off AGND.
The leftover AGND stub next to pad 3 was 0.04 mm from the open OUT-
pad. That stub is gone. DRC is clean at every severity. Assembly BOM
drops J1 (62 parts); jlcpcb_extra.csv still lists C124378 so the
header can be ordered loose.

Co-authored-by: zachrobertson19 <zachrobertson19@gmail.com>
Routing:
- net /Audio/AGND: track 43.1 -> 38.7 mm
Changed lines of the file:
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@@
-	)
-	(segment
-		(start 30.5202 16.2049)
-		(end 30.5202 11.8298)
-		(width 0.15)
-		(locked yes)
-		(layer "F.Cu")
-		(net "/Audio/AGND")
 	)
 	(segment
@@
 		(end 30.5202 16.2049)
 		(width 0.15)
-		(locked yes)
-		(layer "F.Cu")
-		(net "/Audio/AGND")
-	)
-	(segment
-		(start 30.5201 16.2049)
-		(end 30.5202 16.2049)
-		(width 0.15)
