File: hardware/kicad/recorder/mcu_usb.kicad_sch (KiCad schematic)
At the start: 13 parts, among them J1 UART0, J2 USB_C_16P, U1 ESP32-S3-MINI-1U-N8, U7 USBLC6-2SC6

Commit message: Match J1/MK1 schematic BOM flags and refresh the JLCPCB upload set.
Excluding those two from the PCB BOM tripped schematic-parity until the
sheets said in_bom no as well. check_gates is green: DRC clean, 60 SMT
placements, every JLC BOM row has an LCSC code, J1 and MK1 off the machine
files.

Co-authored-by: zachrobertson19 <zachrobertson19@gmail.com>
Parts:
- J1: now left out of the parts list
Changed lines of the file:
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@@
 		(unit 1)
 		(exclude_from_sim no)
-		(in_bom yes)
+		(in_bom no)
 		(on_board yes)
 		(dnp no)
